Commit message: removed static dexmo ref from xacro

File: human_arm_description/model/human_arm.urdf.xacro (robot description, xacro)
@@ -233,10 +233,10 @@
 		</xacro:finger>
 		<!-- Dexmo Ref -->
-		<link name="dexmo_ref"/>
-		<joint name="${joint_prefix}dexmo_ref_static" type="fixed">
-			<parent link="palm_link" />
-			<child link="dexmo_ref"/>
-			<origin xyz="${link_lengths['palm_link_distances']['middle']['x']} 0.0135 ${link_lengths['palm_link_distances']['middle']['z'] - link_lengths['dexmo_ref']}" rpy="0 0 0"/>
-		</joint>
+		<!--<link name="dexmo_ref"/> -->
+		<!--<joint name="${joint_prefix}dexmo_ref_static" type="fixed"> -->
+			<!--<parent link="palm_link" /> -->
+			<!--<child link="dexmo_ref"/> -->
+			<!--<origin xyz="${link_lengths['palm_link_distances']['middle']['x']} 0.0135 ${link_lengths['palm_link_distances']['middle']['z'] - link_lengths['dexmo_ref']}" rpy="0 0 0"/> -->
+		<!--</joint> -->
 	</xacro:macro>
 </robot>
